File: Desk Amplifier.kicad_pcb (KiCad board)
At the start: 2 copper layers, 57 x 81 mm, 37 parts, among them J1 STX-3000, J2 STX-3000, J3 STX-3000, J4 STX-3000, J6 USB4970-00-A, U1 OPA2134, U2 OPA2134

Commit message: fixup routing
Parts:
- moved C9 0.50 mm to (109.8, 124.0)
Routing:
- net Net-(C8-Pad1): track 28.0 -> 28.9 mm
- net Net-(C6-Pad2): track 25.5 -> 24.7 mm
Other:
- board text added: "zot zot zot! github.com/MicahRaney/Desk-Amplifier"
Changed lines of the file:
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@@
 	(footprint "Capacitor_THT:C_Disc_D5.0mm_W2.5mm_P2.50mm"
 		(layer "F.Cu")
-		(at 109.75 123.5)
+		(at 109.75 124)
 		(descr "C, Disc series, Radial, pin pitch=2.50mm, diameter*width=5*2.5mm^2, Capacitor, http://cdn-reichelt.de/documents/datenblatt/B300/DS_KERKO_TC.pdf")
 		(tags "C Disc series Radial pin pitch 2.50mm diameter 5mm width 2.5mm Capacitor")
@@
 		)
 	)
+	(gr_text "zot zot zot!\ngithub.com/MicahRaney/Desk-Amplifier\n"
+		(at 136.5 136.5 0)
+		(layer "B.SilkS")
+		(effects
+			(font
+				(size 1 1)
+				(thickness 0.25)
+				(bold yes)
+			)
+			(justify left bottom mirror)
+		)
+	)
 	(dimension
 		(type orthogonal)
@@
 	)
 	(segment
-		(start 115 123.5)
-		(end 112.25 123.5)
+		(start 115.5 124)
+		(end 112.25 124)
 		(width 0.4)
 		(layer "B.Cu")
@@
 	)
 	(segment
-		(start 112.25 123.5)
-		(end 112.25 120.25)
+		(start 117.19 125.69)
+		(end 115.5 124)
 		(width 0.4)
 		(layer "B.Cu")
@@
 	)
 	(segment
-		(start 117.19 125.69)
-		(end 115 123.5)
+		(start 112.25 124)
+		(end 112.25 120.25)
 		(width 0.4)
 		(layer "B.Cu")
@@
 	)
 	(segment
-		(start 113.62 105.5)
-		(end 120.31 112.19)
+		(start 112.62 104.5)
+		(end 105.75 104.5)
+		(width 0.2)
+		(layer "B.Cu")
+		(net "Net-(C8-Pad1)")
+	)
+	(segment
+		(start 105.75 104.5)
+		(end 105.25 105)
 		(width 0.2)
 		(layer "B.Cu")
@@
 	)
 	(segment
-		(start 105.5 105.5)
-		(end 113.62 105.5)
+		(start 120.31 112.19)
+		(end 112.62 104.5)
 		(width 0.2)
 		(layer "B.Cu")
@@
 	)
 	(segment
-		(start 126.5 103)
+		(start 125.5 98)
 		(end 128.5 101)
 		(width 0.2)
@@
 	)
 	(segment
-		(start 109.5 103)
-		(end 126.5 103)
+		(start 105.5 99)
+		(end 106.5 98)
 		(width 0.2)
 		(layer "B.Cu")
@@
 	)
 	(segment
-		(start 105.5 99)
-		(end 109.5 103)
+		(start 106.5 98)
+		(end 125.5 98)
 		(width 0.2)
 		(layer "B.Cu")
