File: Desk Amplifier.kicad_pcb (KiCad board)
At the start: 2 copper layers, 57 x 81 mm, 37 parts, among them J1 STX-3000, J2 STX-3000, J3 STX-3000, J4 STX-3000, J6 USB4970-00-A, U1 OPA2134, U2 OPA2134

Commit message: fix nets & round corners
Parts:
- H1, H2, H3: footprint MountingHole:MountingHole_2.1mm -> MountingHole:MountingHole_2.5mm
Other:
- outline, holes or cut-outs redrawn
- board text added: "Desk Amp Rev 1.1 Micah Raney micahraney.com 2026"
- board text removed: "Desk Amp Rev 1 Micah Raney micahraney.com 2026"
Changed lines of the file:
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@@
 			)
 		)
-		(property "Datasheet" ""
+		(property "Datasheet" "https://www.digikey.com/en/products/detail/stackpole-electronics-inc/CF14JT10K0/1741265"
 			(at 0 0 0)
 			(layer "F.Fab")
@@
 		)
 	)
-	(footprint "MountingHole:MountingHole_2.1mm"
+	(footprint "MountingHole:MountingHole_2.5mm"
 		(layer "F.Cu")
 		(at 131.5 131.5)
-		(descr "Mounting Hole 2.1mm, no annular, generated by kicad-footprint-generator mountinghole.py")
+		(descr "Mounting Hole 2.5mm, no annular, generated by kicad-footprint-generator mountinghole.py")
 		(tags "mountinghole")
 		(property "Reference" "H1"
-			(at 0 -3.05 0)
+			(at 0 -3.45 0)
 			(layer "F.SilkS")
 			(effects
@@
 		)
 		(property "Value" "MountingHole"
-			(at 0 3.05 0)
+			(at 0 3.45 0)
 			(layer "F.Fab")
 			(effects
@@
 		(fp_circle
 			(center 0 0)
-			(end 2.1 0)
+			(end 2.5 0)
 			(stroke
 				(width 0.15)
@@
 		(fp_circle
 			(center 0 0)
-			(end 2.35 0)
+			(end 2.75 0)
 			(stroke
 				(width 0.05)
@@
 		)
 		(fp_text user "${REFERENCE}"
-			(at 0 0.5 0)
+			(at 0 0 0)
 			(layer "F.Fab")
 			(effects
@@
 		(pad "" np_thru_hole circle
 			(at 0 0)
-			(size 2.1 2.1)
-			(drill 2.1)
+			(size 2.5 2.5)
+			(drill 2.5)
 			(layers "*.Cu" "*.Mask")
 		)
@@
 			)
 		)
-		(property "Datasheet" ""
+		(property "Datasheet" "https://www.digikey.com/en/products/detail/stackpole-electronics-inc/CF14JT10K0/1741265"
 			(at 0 0 0)
 			(layer "F.Fab")
@@
 			)
 		)
-		(property "Datasheet" ""
+		(property "Datasheet" "https://www.digikey.com/en/products/detail/yageo/CFR-25JT-52-5K1/9098642"
 			(at 0 0 0)
 			(layer "F.Fab")
@@
 			)
 		)
-		(property "Datasheet" ""
+		(property "Datasheet" "https://www.digikey.com/en/products/detail/tdk/FG18X5R1E106MRT06/7384735"
 			(at 0 0 180)
 			(layer "F.Fab")
@@
 			)
 		)
-		(property "Datasheet" ""
+		(property "Datasheet" "https://www.digikey.com/en/products/detail/tdk/FG18C0G1H010CNT06/5802778?s=N4IgTCBcDaIGIHECMAOAwgBmQCQ0jaAcgCoYBsIAugL5A"
 			(at 0 0 180)
 			(layer "F.Fab")
@@
 			)
 		)
-		(property "Datasheet" ""
+		(property "Datasheet" "https://www.digikey.com/en/products/detail/tdk/FG18X5R1E106MRT06/7384735"
 			(at 0 0 0)
 			(layer "F.Fab")
@@
 			)
 		)
-		(property "Datasheet" ""
+		(property "Datasheet" "https://www.digikey.com/en/products/detail/tdk/FG18X5R1E106MRT06/7384735"
 			(at 0 0 180)
 			(layer "F.Fab")
@@
 			)
 		)
-		(property "Datasheet" ""
+		(property "Datasheet" "https://www.digikey.com/en/products/detail/tdk/FG18X5R1E106MRT06/7384735"
 			(at 0 0 0)
 			(layer "F.Fab")
@@
 			)
 		)
-		(property "Datasheet" ""
+		(property "Datasheet" "https://www.digikey.com/en/products/detail/tdk/FG18X5R1E106MRT06/7384735"
 			(at 0 0 0)
 			(layer "F.Fab")
@@
 			)
 		)
-		(property "Datasheet" ""
+		(property "Datasheet" "https://www.digikey.com/en/products/detail/tdk/FG18C0G1H010CNT06/5802778?s=N4IgTCBcDaIGIHECMAOAwgBmQCQ0jaAcgCoYBsIAugL5A"
 			(at 0 0 0)
 			(layer "F.Fab")
@@
 			)
 		)
-		(property "Datasheet" ""
+		(property "Datasheet" "https://www.digikey.com/en/products/detail/stackpole-electronics-inc/CF14JT10K0/1741265"
 			(at 0 0 0)
 			(layer "F.Fab")
@@
 			)
 		)
-		(property "Datasheet" ""
+		(property "Datasheet" "https://www.digikey.com/en/products/detail/yageo/CFR-25JT-52-5K1/9098642"
 			(at 0 0 0)
 			(layer "F.Fab")
@@
 			)
 		)
-		(property "Datasheet" ""
+		(property "Datasheet" "https://www.digikey.com/en/products/detail/stackpole-electronics-inc/CF14JT1M00/1741316"
 			(at 0 0 0)
 			(layer "F.Fab")
@@
 			)
 		)
-		(property "Datasheet" ""
+		(property "Datasheet" "https://www.digikey.com/en/products/detail/stackpole-electronics-inc/CF14JT10K0/1741265"
 			(at 0 0 0)
 			(layer "F.Fab")
@@
 			)
 		)
-		(property "Datasheet" ""
+		(property "Datasheet" "https://www.digikey.com/en/products/detail/stackpole-electronics-inc/CF14JT10K0/1741265"
 			(at 0 0 0)
 			(layer "F.Fab")
@@
 			)
 		)
-		(property "Datasheet" ""
+		(property "Datasheet" "https://www.digikey.com/en/products/detail/tdk/FG18X5R1E106MRT06/7384735"
 			(at 0 0 0)
 			(layer "F.Fab")
@@
 			)
 		)
-		(property "Datasheet" ""
+		(property "Datasheet" "https://www.digikey.com/en/products/detail/stackpole-electronics-inc/CF14JT10K0/1741265"
 			(at 0 0 0)
 			(layer "F.Fab")
@@
 		)
 	)
-	(footprint "MountingHole:MountingHole_2.1mm"
+	(footprint "MountingHole:MountingHole_2.5mm"
 		(layer "F.Cu")
 		(at 86.5 119)
-		(descr "Mounting Hole 2.1mm, no annular, generated by kicad-footprint-generator mountinghole.py")
+		(descr "Mounting Hole 2.5mm, no annular, generated by kicad-footprint-generator mountinghole.py")
 		(tags "mountinghole")
 		(property "Reference" "H3"
-			(at 3.5 -0.5 0)
+			(at 0 -3.45 0)
 			(layer "F.SilkS")
 			(effects
@@
 		)
 		(property "Value" "MountingHole"
-			(at 0 3.05 0)
+			(at 0 3.45 0)
 			(layer "F.Fab")
 			(effects
@@
 		(fp_circle
 			(center 0 0)
-			(end 2.1 0)
+			(end 2.5 0)
 			(stroke
 				(width 0.15)
@@
 		(fp_circle
 			(center 0 0)
-			(end 2.35 0)
+			(end 2.75 0)
 			(stroke
 				(width 0.05)
@@
 		(pad "" np_thru_hole circle
 			(at 0 0)
-			(size 2.1 2.1)
-			(drill 2.1)
+			(size 2.5 2.5)
+			(drill 2.5)
 			(layers "*.Cu" "*.Mask")
 		)
@@
 			)
 		)
-		(property "Datasheet" ""
+		(property "Datasheet" "https://www.digikey.com/en/products/detail/stackpole-electronics-inc/CF14JT1M00/1741316"
 			(at 0 0 0)
 			(layer "F.Fab")
@@
 			)
 		)
-		(property "Datasheet" ""
+		(property "Datasheet" "https://www.digikey.com/en/products/detail/stackpole-electronics-inc/CF14JT10K0/1741265"
 			(at 0 0 0)
 			(layer "F.Fab")
@@
 		)
 	)
-	(footprint "MountingHole:MountingHole_2.1mm"
+	(footprint "MountingHole:MountingHole_2.5mm"
 		(layer "F.Cu")
 		(at 111.5 62.5)
-		(descr "Mounting Hole 2.1mm, no annular, generated by kicad-footprint-generator mountinghole.py")
+		(descr "Mounting Hole 2.5mm, no annular, generated by kicad-footprint-generator mountinghole.py")
 		(tags "mountinghole")
 		(property "Reference" "H2"
-			(at 0 -3.05 0)
+			(at 0 -3.45 0)
 			(layer "F.SilkS")
 			(effects
@@
 		)
 		(property "Value" "MountingHole"
-			(at 0 3.05 0)
+			(at 0 3.45 0)
 			(layer "F.Fab")
 			(effects
@@
 		(fp_circle
 			(center 0 0)
-			(end 2.1 0)
+			(end 2.5 0)
 			(stroke
 				(width 0.15)
@@
 		(fp_circle
 			(center 0 0)
-			(end 2.35 0)
+			(end 2.75 0)
 			(stroke
 				(width 0.05)
@@
 		)
 		(fp_text user "${REFERENCE}"
-			(at 0 0.5 0)
+			(at 0 0 0)
 			(layer "F.Fab")
 			(effects
@@
 		(pad "" np_thru_hole circle
 			(at 0 0)
-			(size 2.1 2.1)
-			(drill 2.1)
+			(size 2.5 2.5)
+			(drill 2.5)
 			(layers "*.Cu" "*.Mask")
 		)
@@
 			)
 		)
-		(property "Datasheet" ""
+		(property "Datasheet" "https://www.digikey.com/en/products/detail/stackpole-electronics-inc/CF14JT10K0/1741265"
 			(at 0 0 0)
 			(layer "F.Fab")
@@
 			)
 		)
-		(property "Datasheet" ""
+		(property "Datasheet" "https://www.digikey.com/en/products/detail/tdk/FG18X5R1E106MRT06/7384735"
 			(at 0 0 0)
 			(layer "F.Fab")
@@
 			)
 		)
-		(property "Datasheet" ""
+		(property "Datasheet" "https://www.digikey.com/en/products/detail/tdk/FG18X5R1E106MRT06/7384735"
 			(at 0 0 0)
 			(layer "F.Fab")
@@
 			)
 		)
-		(property "Datasheet" ""
+		(property "Datasheet" "https://www.digikey.com/en/products/detail/stackpole-electronics-inc/CF14JT10K0/1741265"
 			(at 0 0 0)
 			(layer "F.Fab")
@@
 			)
 		)
-		(property "Datasheet" ""
+		(property "Datasheet" "https://www.digikey.com/en/products/detail/stackpole-electronics-inc/CF14JT10K0/1741265"
 			(at 0 0 0)
 			(layer "F.Fab")
@@
 		)
 	)
-	(gr_rect
-		(start 80.5 56.5)
-		(end 137.5 137.5)
+	(gr_arc
+		(start 80.5 58)
+		(mid 80.93934 56.93934)
+		(end 82 56.5)
+		(stroke
+			(width 0.05)
+			(type default)
+		)
+		(layer "Edge.Cuts")
+	)
+	(gr_line
+		(start 80.5 136.5)
+		(end 80.5 58)
+		(stroke
+			(width 0.05)
+			(type default)
+		)
+		(layer "Edge.Cuts")
+	)
+	(gr_arc
+		(start 81.5 137.5)
+		(mid 80.792893 137.207107)
+		(end 80.5 136.5)
+		(stroke
+			(width 0.05)
+			(type default)
+		)
+		(layer "Edge.Cuts")
+	)
+	(gr_line
+		(start 82 56.5)
+		(end 136.5 56.5)
+		(stroke
+			(width 0.05)
+			(type default)
+		)
+		(layer "Edge.Cuts")
+	)
+	(gr_arc
+		(start 136.5 56.5)
+		(mid 137.207107 56.792893)
+		(end 137.5 57.5)
+		(stroke
+			(width 0.05)
+			(type default)
+		)
+		(layer "Edge.Cuts")
+	)
+	(gr_line
+		(start 136.5 137.5)
+		(end 81.5 137.5)
+		(stroke
+			(width 0.05)
+			(type default)
+		)
+		(layer "Edge.Cuts")
+	)
+	(gr_line
+		(start 137.5 57.5)
+		(end 137.5 136.5)
+		(stroke
+			(width 0.05)
+			(type default)
+		)
+		(layer "Edge.Cuts")
+	)
+	(gr_arc
+		(start 137.5 136.5)
+		(mid 137.207107 137.207107)
+		(end 136.5 137.5)
 		(stroke
 			(width 0.05)
 			(type default)
 		)
-		(fill no)
 		(layer "Edge.Cuts")
 	)
-	(gr_text "Desk Amp Rev 1\nMicah Raney\nmicahraney.com\n2026"
-		(at 124 123 0)
+	(gr_text "Desk Amp Rev 1.1\nMicah Raney\nmicahraney.com\n2026"
+		(at 122.5 123.5 0)
 		(layer "F.SilkS")
 		(effects
@@
 		(layer "User.1")
 		(pts
-			(xy 128.5 66) (xy 131.5 56.5)
+			(xy 128.5 66) (xy 137.5 56.5)
 		)
 		(height 34.5)
@@
 		(polygon
 			(pts
-				(xy 80.5 56.5) (xy 137 56.5) (xy 137 137.5) (xy 80.5 137.5)
+				(xy 80.5 56.5) (xy 137.5 56.5) (xy 137.5 137.5) (xy 80.5 137.5)
 			)
 		)
@@
 		(polygon
 			(pts
-				(xy 80.5 56.5) (xy 137 56.5) (xy 137 137.5) (xy 80.5 137.5)
+				(xy 80.5 56.5) (xy 137.5 56.5) (xy 137.5 137.5) (xy 80.5 137.5)
 			)
 		)
